File: board/modules/clocking/clocking.kicad_sch (KiCad schematic)
At the start: 0 parts

Commit message: 1. Update to Local Symbol Library 2. Clocking Module Schematic
Parts:
- added C1: 1u, symbol 8bitcomp:Cap
- added C2, C3, C4, C6, C7, C8: 100n, symbol 8bitcomp:Cap
- added C5: 10u, symbol 8bitcomp:Cap-Polarized
- added C9: 100u, symbol 8bitcomp:Cap-Polarized
- added D1: 1N4148, symbol 8bitcomp:Diode
- added D2: GREEN, symbol 8bitcomp:LED
- added D3: RED, symbol 8bitcomp:LED
- added D4: WHITE, symbol 8bitcomp:LED
- added R1, R10, R2, R3, R4, R8, R9: 1k, symbol 8bitcomp:Res
- added R5, R6: 10k, symbol 8bitcomp:Res
- added R7: 100k, symbol 8bitcomp:Res
- added RV1: 1Meg, symbol 8bitcomp:R_Pot
- added SW1: CLK, symbol 8bitcomp:TacatileSW
- added SW2: SEL, symbol 8bitcomp:TacatileSW
- added TP1: VCC, symbol 8bitcomp:TestPoint
- added TP2: GND, symbol 8bitcomp:TestPoint
- added TP3: HALT, symbol 8bitcomp:TestPoint
- added TP4: Output, symbol 8bitcomp:TestPoint
- added U1, U2, U3, U4: NE555D, Package_SO:SOIC-8_3.9x4.9mm_P1.27mm, symbol 8bitcomp:NE555D
- added U5: 7404, Package_SO:SOIC-14_3.9x8.7mm_P1.27mm, symbol 8bitcomp:7404
- added U6, U7, U8: 7400, Package_SO:SOIC-14_3.9x8.7mm_P1.27mm, symbol 8bitcomp:7400
Connections:
- new net: U5.4, U7.13
- new net: R5.2, R6.1, SW2.2, U3.2 (TR), U3.6 (THR)
- new net: D2.2 (A), R8.2, U4.3 (Q), U5.11, U8.2
- new net: U7.9, U8.3
- new net: U5.8, U6.9
- new net: R7.1, U3.3 (Q), U5.9, U6.12
- new net: D1.1 (K), R2.2, RV1.1, U1.2 (TR), U1.6 (THR)
- new net: U1.4 (R), U7.3
- new net: C2.1, U1.5 (CV)
- new net: D1.2 (A), R1.2, R2.1, U1.7 (DIS)
- new net: C3.1, R4.2, U2.6 (THR), U2.7 (DIS)
- new net: D4.1 (K), R10.1
- new net: D4.2 (A), TP4.1, U7.8
- new net: U7.10, U7.6
- new net: U4.2 (TR), U6.11
- new net: U4.4 (R), U6.8
- new net: C7.1, U4.5 (CV)
- new net: D3.1 (K), R8.1
- new net: R3.2, SW1.2, U2.2 (TR)
- new net: U2.4 (R), U6.6
- new net: U5.6, U6.10, U6.13
- new net: C6.1, U3.5 (CV)
- new net: U5.2, U7.12
- new net: D2.1 (K), R9.1
- new net: U5.5, U7.11
- new net: C1.1, RV1.2, RV1.3
- new net: U5.10, U7.4
- new net: C5.1, R7.2, SW2.1
- new net: C4.1, U2.5 (CV)
- new net +5V: C8.1, C9.1, D3.2 (A), R1.1, R3.1, R4.1, R5.1, TP1.1, U1.8 (VCC), U2.8 (VCC), U3.4 (R), U3.8 (VCC), U4.8 (VCC), U5.14 (VCC), U6.14 (VCC), U7.14 (VCC)
- new net FRC: U1.3 (Q), U5.1, U8.1
- new net FRC_rst_sync: U7.1
- new net GND: C1.2, C2.2, C3.2, C4.2, C5.2, C6.2, C7.2, C8.2, C9.2, R10.2, R6.2, R9.2, SW1.1, TP2.1, U1.1 (GND), U2.1 (GND), U3.1 (GND), U4.1 (GND), U5.7 (GND), U6.7 (GND), U7.7 (GND)
- new net HALT: TP3.1, U6.5, U7.2
- new net MCC: U2.3 (Q), U5.3, U7.5
- new net MCC_rst_sync: U6.4
- no-connect marks 0 -> 3
Other:
- note added: "Astable"
- note added: "Clock Source = Free Running"
- note added: "Clock Source = Manual"
- note added: "Clock Status"
- note added: "Decap"
- note added: "Monostable"
- note added: "Selector"
- note added: "Syncronizer Latch"
