File: board/modules/clocking/clocking.kicad_sch (KiCad schematic)
At the start: 38 parts, among them SW1 CLK, SW2 SEL, U1 NE555D, U2 NE555D, U3 NE555D, U4 NE555D, U5 7404, U6 7400, U7 7400, U8 7400

Commit message: Updating Footprint Mapping
Parts:
- C1, C2, C3, C4, C6, C7, C8: footprint (none) -> 8bitcomp:C_0603_1608Metric_Pad1.08x0.95mm_HandSolder
- C5, C9: footprint (none) -> 8bitcomp:CP_EIA-3216-18_Kemet-A
- D1: footprint (none) -> 8bitcomp:D_SOD-323
- D2, D3, D4: footprint (none) -> 8bitcomp:LED_0603_1608Metric
- R1, R10, R2, R3, R4, R5, R6, R7, R8, R9: footprint (none) -> 8bitcomp:R_0603_1608Metric_Pad0.98x0.95mm_HandSolder
- RV1: footprint (none) -> 8bitcomp:Potentiometer_Piher_PT-15-V15_Vertical_Hole
- SW1, SW2: footprint (none) -> 8bitcomp:SW_SPST_EVQPE1
- TP1, TP2, TP3, TP4: footprint (none) -> 8bitcomp:TestPoint_Pad_D3.0mm
- U1, U2, U3, U4: footprint Package_SO:SOIC-8_3.9x4.9mm_P1.27mm -> 8bitcomp:SOIC-8_3.9x4.9mm_P1.27mm
- U5, U6, U7, U8: footprint Package_SO:SOIC-14_3.9x8.7mm_P1.27mm -> 8bitcomp:SOIC-14_3.9x8.7mm_P1.27mm
Changed lines of the file:
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@@
 	(label "HALT"
 		(at 71.12 29.21 180)
-		(fields_autoplaced yes)
 		(effects
 			(font
@@
 	(label "HALT"
 		(at 142.24 30.48 270)
-		(fields_autoplaced yes)
 		(effects
 			(font
@@
 	(label "FRC"
 		(at 168.91 111.76 0)
-		(fields_autoplaced yes)
 		(effects
 			(font
@@
 	(label "MCC"
 		(at 158.75 62.23 180)
-		(fields_autoplaced yes)
 		(effects
 			(font
@@
 	(label "FRC"
 		(at 46.99 154.94 0)
-		(fields_autoplaced yes)
 		(effects
 			(font
@@
 	(label "MCC"
 		(at 46.99 167.64 0)
-		(fields_autoplaced yes)
 		(effects
 			(font
@@
 	(label "MCC"
 		(at 168.91 130.81 0)
-		(fields_autoplaced yes)
 		(effects
 			(font
@@
 	(label "MCC_rst_sync"
 		(at 161.29 31.75 180)
-		(fields_autoplaced yes)
 		(effects
 			(font
@@
 	(label "FRC_rst_sync"
 		(at 110.49 31.75 180)
-		(fields_autoplaced yes)
 		(effects
 			(font
@@
 	(label "HALT"
 		(at 91.44 30.48 270)
-		(fields_autoplaced yes)
 		(effects
 			(font
@@
 	(label "FRC"
 		(at 107.95 62.23 180)
-		(fields_autoplaced yes)
 		(effects
 			(font
@@
 			)
 		)
-		(property "Footprint" "Package_SO:SOIC-14_3.9x8.7mm_P1.27mm"
+		(property "Footprint" "8bitcomp:SOIC-14_3.9x8.7mm_P1.27mm"
 			(at 63.5 167.64 0)
 			(effects
@@
 			)
 		)
-		(property "Footprint" ""
+		(property "Footprint" "8bitcomp:R_0603_1608Metric_Pad0.98x0.95mm_HandSolder"
 			(at 62.23 133.35 0)
 			(effects
@@
 			)
 		)
-		(property "Footprint" "Package_SO:SOIC-14_3.9x8.7mm_P1.27mm"
+		(property "Footprint" "8bitcomp:SOIC-14_3.9x8.7mm_P1.27mm"
 			(at 180.34 114.3 0)
 			(effects
@@
 			)
 		)
-		(property "Footprint" "Package_SO:SOIC-14_3.9x8.7mm_P1.27mm"
+		(property "Footprint" "8bitcomp:SOIC-14_3.9x8.7mm_P1.27mm"
 			(at 102.87 106.68 0)
 			(effects
@@
 			)
 		)
-		(property "Footprint" "Package_SO:SOIC-8_3.9x4.9mm_P1.27mm"
+		(property "Footprint" "8bitcomp:SOIC-8_3.9x4.9mm_P1.27mm"
 			(at 92.456 80.518 0)
 			(effects
@@
 			)
 		)
-		(property "Footprint" ""
+		(property "Footprint" "8bitcomp:C_0603_1608Metric_Pad1.08x0.95mm_HandSolder"
 			(at 128.27 80.01 0)
 			(effects
@@
 			)
 		)
-		(property "Footprint" ""
+		(property "Footprint" "8bitcomp:CP_EIA-3216-18_Kemet-A"
 			(at 181.61 40.64 0)
 			(effects
@@
 			)
 		)
-		(property "Footprint" ""
+		(property "Footprint" "8bitcomp:R_0603_1608Metric_Pad0.98x0.95mm_HandSolder"
 			(at 207.01 140.97 0)
 			(effects
@@
 			)
 		)
-		(property "Footprint" ""
+		(property "Footprint" "8bitcomp:R_0603_1608Metric_Pad0.98x0.95mm_HandSolder"
 			(at 128.27 54.61 0)
 			(effects
@@
 			)
 		)
-		(property "Footprint" ""
+		(property "Footprint" "8bitcomp:C_0603_1608Metric_Pad1.08x0.95mm_HandSolder"
 			(at 93.98 80.01 0)
 			(effects
@@
 			)
 		)
-		(property "Footprint" ""
+		(property "Footprint" "8bitcomp:TestPoint_Pad_D3.0mm"
 			(at 209.55 125.73 0)
 			(effects
@@
 			)
 		)
-		(property "Footprint" "Package_SO:SOIC-14_3.9x8.7mm_P1.27mm"
+		(property "Footprint" "8bitcomp:SOIC-14_3.9x8.7mm_P1.27mm"
 			(at 198.12 120.65 0)
 			(effects
@@
 			)
 		)
-		(property "Footprint" ""
+		(property "Footprint" "8bitcomp:TestPoint_Pad_D3.0mm"
 			(at 203.2 59.69 0)
 			(effects
@@
 			)
 		)
-		(property "Footprint" ""
+		(property "Footprint" "8bitcomp:R_0603_1608Metric_Pad0.98x0.95mm_HandSolder"
 			(at 73.66 54.61 0)
 			(effects
@@
 			)
 		)
-		(property "Footprint" "Package_SO:SOIC-8_3.9x4.9mm_P1.27mm"
+		(property "Footprint" "8bitcomp:SOIC-8_3.9x4.9mm_P1.27mm"
 			(at 139.446 144.018 0)
 			(effects
@@
 			)
 		)
-		(property "Footprint" ""
+		(property "Footprint" "8bitcomp:R_0603_1608Metric_Pad0.98x0.95mm_HandSolder"
 			(at 154.94 111.76 0)
 			(effects
@@
 			)
 		)
-		(property "Footprint" "Package_SO:SOIC-14_3.9x8.7mm_P1.27mm"
+		(property "Footprint" "8bitcomp:SOIC-14_3.9x8.7mm_P1.27mm"
 			(at 184.15 69.85 0)
 			(effects
@@
 			)
 		)
-		(property "Footprint" ""
+		(property "Footprint" "8bitcomp:R_0603_1608Metric_Pad0.98x0.95mm_HandSolder"
 			(at 123.19 54.61 0)
 			(effects
@@
 			)
 		)
-		(property "Footprint" "Package_SO:SOIC-14_3.9x8.7mm_P1.27mm"
+		(property "Footprint" "8bitcomp:SOIC-14_3.9x8.7mm_P1.27mm"
 			(at 144.78 40.64 0)
 			(effects
@@
 			)
 		)
-		(property "Footprint" ""
+		(property "Footprint" "8bitcomp:TestPoint_Pad_D3.0mm"
 			(at 67.31 24.13 0)
 			(effects
@@
 			)
 		)
-		(property "Footprint" ""
+		(property "Footprint" "8bitcomp:D_SOD-323"
 			(at 67.31 62.23 90)
 			(effects
@@
 			)
 		)
-		(property "Footprint" "Package_SO:SOIC-14_3.9x8.7mm_P1.27mm"
+		(property "Footprint" "8bitcomp:SOIC-14_3.9x8.7mm_P1.27mm"
 			(at 118.11 109.22 0)
 			(effects
@@
 			)
 		)
-		(property "Footprint" ""
+		(property "Footprint" "8bitcomp:C_0603_1608Metric_Pad1.08x0.95mm_HandSolder"
 			(at 81.28 143.51 0)
 			(effects
@@
 			)
 		)
-		(property "Footprint" ""
+		(property "Footprint" "8bitcomp:C_0603_1608Metric_Pad1.08x0.95mm_HandSolder"
 			(at 140.97 143.51 0)
 			(effects
@@
 			)
 		)
-		(property "Footprint" "Package_SO:SOIC-14_3.9x8.7mm_P1.27mm"
+		(property "Footprint" "8bitcomp:SOIC-14_3.9x8.7mm_P1.27mm"
 			(at 63.5 154.94 0)
 			(effects
@@
 			)
 		)
-		(property "Footprint" "Package_SO:SOIC-14_3.9x8.7mm_P1.27mm"
+		(property "Footprint" "8bitcomp:SOIC-14_3.9x8.7mm_P1.27mm"
 			(at 118.11 132.08 0)
 			(effects
@@
 			)
 		)
-		(property "Footprint" ""
+		(property "Footprint" "8bitcomp:R_0603_1608Metric_Pad0.98x0.95mm_HandSolder"
 			(at 154.94 140.97 0)
 			(effects
@@
 			)
 		)
-		(property "Footprint" "Package_SO:SOIC-14_3.9x8.7mm_P1.27mm"
+		(property "Footprint" "8bitcomp:SOIC-14_3.9x8.7mm_P1.27mm"
 			(at 99.06 161.29 0)
 			(effects
@@
 			)
 		)
-		(property "Footprint" ""
+		(property "Footprint" "8bitcomp:TestPoint_Pad_D3.0mm"
 			(at 203.2 66.04 0)
 			(effects
@@
 			)
 		)
-		(property "Footprint" "Package_SO:SOIC-8_3.9x4.9mm_P1.27mm"
+		(property "Footprint" "8bitcomp:SOIC-8_3.9x4.9mm_P1.27mm"
 			(at 79.756 144.018 0)
 			(effects
@@
 			)
 		)
-		(property "Footprint" ""
+		(property "Footprint" "8bitcomp:C_0603_1608Metric_Pad1.08x0.95mm_HandSolder"
 			(at 73.66 80.01 0)
 			(effects
@@
 			)
 		)
-		(property "Footprint" "Package_SO:SOIC-14_3.9x8.7mm_P1.27mm"
+		(property "Footprint" "8bitcomp:SOIC-14_3.9x8.7mm_P1.27mm"
 			(at 180.34 128.27 0)
 			(effects
@@
 			)
 		)
-		(property "Footprint" "Package_SO:SOIC-14_3.9x8.7mm_P1.27mm"
+		(property "Footprint" "8bitcomp:SOIC-14_3.9x8.7mm_P1.27mm"
 			(at 193.04 69.85 0)
 			(effects
@@
 			)
 		)
-		(property "Footprint" "Package_SO:SOIC-14_3.9x8.7mm_P1.27mm"
+		(property "Footprint" "8bitcomp:SOIC-14_3.9x8.7mm_P1.27mm"
 			(at 175.26 69.85 0)
 			(effects
@@
 			)
 		)
-		(property "Footprint" "Package_SO:SOIC-14_3.9x8.7mm_P1.27mm"
+		(property "Footprint" "8bitcomp:SOIC-14_3.9x8.7mm_P1.27mm"
 			(at 165.1 125.73 0)
 			(effects
@@
 			)
 		)
-		(property "Footprint" ""
+		(property "Footprint" "8bitcomp:R_0603_1608Metric_Pad0.98x0.95mm_HandSolder"
 			(at 62.23 125.73 0)
 			(effects
@@
 			)
 		)
-		(property "Footprint" ""
+		(property "Footprint" "8bitcomp:SW_SPST_EVQPE1"
 			(at 54.61 124.46 0)
 			(effects
@@
 			)
 		)
-		(property "Footprint" ""
+		(property "Footprint" "8bitcomp:SW_SPST_EVQPE1"
 			(at 118.11 77.47 0)
 			(effects
@@
 			)
 		)
-		(property "Footprint" ""
+		(property "Footprint" "8bitcomp:LED_0603_1608Metric"
 			(at 154.94 133.35 90)
 			(effects
@@
 			)
 		)
-		(property "Footprint" "Package_SO:SOIC-14_3.9x8.7mm_P1.27mm"
+		(property "Footprint" "8bitcomp:SOIC-14_3.9x8.7mm_P1.27mm"
 			(at 83.82 161.29 0)
 			(effects
@@
 			)
 		)
-		(property "Footprint" "Package_SO:SOIC-14_3.9x8.7mm_P1.27mm"
+		(property "Footprint" "8bitcomp:SOIC-14_3.9x8.7mm_P1.27mm"
 			(at 93.98 40.64 0)
 			(effects
@@
 			)
 		)
-		(property "Footprint" ""
+		(property "Footprint" "8bitcomp:C_0603_1608Metric_Pad1.08x0.95mm_HandSolder"
 			(at 176.53 40.64 0)
 			(effects
@@
 			)
 		)
-		(property "Footprint" ""
+		(property "Footprint" "8bitcomp:LED_0603_1608Metric"
 			(at 154.94 106.68 90)
 			(effects
@@
 			)
 		)
-		(property "Footprint" ""
+		(property "Footprint" "8bitcomp:C_0603_1608Metric_Pad1.08x0.95mm_HandSolder"
 			(at 144.78 80.01 0)
 			(effects
@@
 			)
 		)
-		(property "Footprint" ""
+		(property "Footprint" "8bitcomp:R_0603_1608Metric_Pad0.98x0.95mm_HandSolder"
 			(at 73.66 62.23 0)
 			(effects
@@
 			)
 		)
-		(property "Footprint" "Package_SO:SOIC-8_3.9x4.9mm_P1.27mm"
+		(property "Footprint" "8bitcomp:SOIC-8_3.9x4.9mm_P1.27mm"
 			(at 143.256 80.518 0)
 			(effects
@@
 			)
 		)
-		(property "Footprint" ""
+		(property "Footprint" "8bitcomp:Potentiometer_Piher_PT-15-V15_Vertical_Hole"
 			(at 73.66 69.85 0)
 			(effects
@@
 			)
 		)
-		(property "Footprint" ""
+		(property "Footprint" "8bitcomp:CP_EIA-3216-18_Kemet-A"
 			(at 48.26 133.35 0)
 			(effects
@@
 			)
 		)
-		(property "Footprint" ""
+		(property "Footprint" "8bitcomp:R_0603_1608Metric_Pad0.98x0.95mm_HandSolder"
 			(at 44.45 129.54 0)
 			(effects
@@
 			)
 		)
-		(property "Footprint" ""
+		(property "Footprint" "8bitcomp:LED_0603_1608Metric"
 			(at 207.01 133.35 90)
 			(effects

Commit message: Updating Schemtic
Parts:
- removed U8: 7400, 8bitcomp:SOIC-14_3.9x8.7mm_P1.27mm, symbol 8bitcomp:7400
- added unit 1 of U6
- D1: footprint 8bitcomp:D_SOD-323 -> 8bitcomp:SOIC-8_3.9x4.9mm_P1.27mm
- U1, U2, U3, U4: footprint 8bitcomp:SOIC-8_3.9x4.9mm_P1.27mm -> Package_SO:SOIC-8_3.9x4.9mm_P1.27mm
Connections:
- net FRC: now also U6.1
- net FRC_rst_sync: now also U7.9, U6.3
- net MCC_rst_sync: now also U7.10, U7.6
- net at D2.2 (A), R8.2, U4.3 (Q)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: now also U6.2
Other:
- moved on the sheet: C5, C6, C7, D2, D3, D4, R10, R5, R6, R7, R8, R9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
