File: board/modules/clocking/clocking.kicad_sch (KiCad schematic)
At the start: 37 parts, among them SW1 CLK, SW2 SEL, U1 NE555D, U2 NE555D, U3 NE555D, U4 NE555D, U5 7404, U6 7400, U7 7400

Commit message: Correction in Astable
Parts:
- added U10, U9: 74LS377, symbol 74xx:74LS377
- added unit 6 of U5
- added U8: IS62C256AL, Package_SO:SOP-28_8.4x18.16mm_P1.27mm, symbol Memory_RAM:IS62C256AL
- D1: footprint 8bitcomp:SOIC-8_3.9x4.9mm_P1.27mm -> 8bitcomp:D_SOD-323
- SW1, SW2: footprint 8bitcomp:SW_SPST_EVQPE1 -> 8bitcomp:SW_Tactile_SPST_NO_Straight_CK_PTS636Sx25SMTRLFS
Connections:
- net GND: now also U8.20 (~{CE})
- net at D1.1 (K), R2.2, RV1.1: no longer U1.2 (TR), U1.6 (THR)
- net at C1.1, RV1.2, RV1.3: now also U1.2 (TR), U1.6 (THR)
- new net: U10.11 (CP), U9.11 (CP)
- new net A0: U8.10 (A0), U9.2 (Q0)
- new net A1: U8.9 (A1), U9.5 (Q1)
- new net A10: U10.6 (Q2), U8.21 (A10)
- new net A11: U10.9 (Q3), U8.23 (A11)
- new net A12: U10.12 (Q4), U8.2 (A12)
- new net A13: U10.15 (Q5), U8.26 (A13)
- new net A14: U10.16 (Q6), U8.1 (A14)
- new net A2: U8.8 (A2), U9.6 (Q2)
- new net A3: U8.7 (A3), U9.9 (Q3)
- new net A4: U8.6 (A4), U9.12 (Q4)
- new net A5: U8.5 (A5), U9.15 (Q5)
- new net A6: U8.4 (A6), U9.16 (Q6)
- new net A7: U8.3 (A7), U9.19 (Q7)
- new net A8: U10.2 (Q0), U8.25 (A8)
- new net A9: U10.5 (Q1), U8.24 (A9)
- new net D0: U10.3 (D0), U9.3 (D0)
- new net D1: U10.4 (D1), U9.4 (D1)
- new net D2: U10.7 (D2), U9.7 (D2)
- new net D3: U10.8 (D3), U9.8 (D3)
- new net D4: U10.13 (D4), U9.13 (D4)
- new net D5: U10.14 (D5), U9.14 (D5)
- new net D6: U10.17 (D6), U9.17 (D6)
- new net D7: U10.18 (D7), U9.18 (D7)
- new net MHI: U10.1 (~{E})
- new net MLI: U9.1 (~{E})
- no-connect marks 3 -> 6
Other:
- moved on the sheet: C1, C2, C3, C4, C5, C6, C7, C8, C9, D1, D2, D3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

Commit message: New PDF Dump of schematic
Parts:
- removed U10, U9: 74LS377, symbol 74xx:74LS377
- removed U8: IS62C256AL, Package_SO:SOP-28_8.4x18.16mm_P1.27mm, symbol Memory_RAM:IS62C256AL
Connections:
- no-connect marks 6 -> 5
